File: sao-wall-tile/sao-wall-tile.kicad_pcb (KiCad board)
At the start: 2 copper layers, 100 x 86.5 mm, 19 parts, among them J1 Power In, J2 Power Out, J3 Power Out, J4 Conn_02x03_Odd_Even, J5 Conn_02x03_Odd_Even, J6 Conn_02x03_Odd_Even, J7 Conn_02x03_Odd_Even

Commit message: Move GPIO pins, update from more review, enhance labels, update renders
Parts:
- removed R7, R8: 5.1K, Resistor_SMD:R_0805_2012Metric_Pad1.20x1.40mm_HandSolder
- added R4: 5.1K, Resistor_SMD:R_0805_2012Metric_Pad1.20x1.40mm_HandSolder, B.Cu at (128.2, 125.0)
- added R5: 5.1K, Resistor_SMD:R_0805_2012Metric_Pad1.20x1.40mm_HandSolder, B.Cu at (122.8, 125.0)
- moved C1 1.27 mm to (108.8, 80.5)
- moved R1 1.03 mm to (107.8, 87.8)
Connections:
- A1 pad 11: unconnected-(A1-GPIO8-Pad11) -> /SAO4_GPIO1
- A1 pad 12: unconnected-(A1-GPIO9-Pad12) -> /SAO4_GPIO2
- A1 pad 19: /SAO4_GPIO1 -> unconnected-(A1-GPIO14-Pad19)
- A1 pad 20: /SAO4_GPIO2 -> unconnected-(A1-GPIO15-Pad20)
Routing:
- net /SAO4_GPIO1: track 33.9 -> 51.5 mm
- net /SAO4_GPIO2: track 36.3 -> 52.0 mm
- net +5V: track 139.8 -> 138.9 mm
- net /EN_3V3: track 9.42 -> 10.1 mm
- net GND: vias 11 -> 14
Other:
- board text added: "GPIO1 SDA 3v3 GPIO2 SCL GND PicoGP0-UART0TX PicoGP1-UART0RX"
- board text added: "GPIO1 SDA 3v3 GPIO2 SCL GND PicoGP19 PicoGP18"
- board text added: "PicoGP14-UART1TX PicoGP15-UART1RX GPIO1 SDA 3v3 GPIO2 SCL GND"
- board text added: "PicoGP16-UART0RX PicoGP17-UART0TX GPIO1 SDA 3v3 GPIO2 SCL GND"
- board text removed: "GPIO1 SDA 3v3 GPIO2 SCL GND"
